Commit message: Amyr Lourensz 2:14 PM / 14:14 2026-06-09
Heb Lite 6 werkcell enviroment en Rviz configuratie

[Toegevoegd: volledige digitale werkomgeving voor de UFACTORY Lite 6, inclusief tafel, werkplatform, montageplaat, stoel, RViz-configuraties, launchbestand en bijbehorende pakketinstellingen.]

File: src/a2_workcell_description/urdf/workcell.urdf.xacro (robot description, xacro)
@@ -2,25 +2,428 @@
 <robot xmlns:xacro="http://www.ros.org/wiki/xacro"
        name="a2_workcell">
+  <!-- ====================================================== -->
+  <!-- AFMETINGEN IN METERS                                   -->
+  <!-- ====================================================== -->
+  <!-- Hoofdtafel -->
+  <xacro:property name="table_length" value="1.60"/>
+  <xacro:property name="table_depth" value="0.80"/>
+  <xacro:property name="table_top_thickness" value="0.025"/>
+  <xacro:property name="table_leg_height" value="0.725"/>
+  <xacro:property name="table_leg_size" value="0.032"/>
+  <xacro:property name="table_leg_edge_offset" value="0.10"/>
+  <!-- Verhoogd robotwerkplatform -->
+  <xacro:property name="platform_length" value="0.80"/>
+  <xacro:property name="platform_depth" value="0.60"/>
+  <xacro:property name="platform_thickness" value="0.019"/>
+  <!-- Tijdelijke breedte van de steunpoten -->
+  <xacro:property name="support_size_x" value="0.060"/>
+  <xacro:property name="support_size_y" value="0.060"/>
+  <xacro:property name="support_height" value="0.040"/>
+  <!-- Metalen plaat onder de Lite 6 -->
+  <xacro:property name="mount_plate_length" value="0.185"/>
+  <xacro:property name="mount_plate_depth" value="0.130"/>
+  <xacro:property name="mount_plate_thickness" value="0.005"/>
+  <!-- Stoel -->
+  <xacro:property name="chair_width" value="0.45"/>
+  <xacro:property name="chair_depth" value="0.45"/>
+  <xacro:property name="chair_seat_thickness" value="0.030"/>
+  <xacro:property name="chair_leg_height" value="0.450"/>
+  <xacro:property name="chair_leg_size" value="0.030"/>
+  <xacro:property name="chair_back_height" value="0.450"/>
+  <xacro:property name="chair_back_thickness" value="0.025"/>
+  <!-- ====================================================== -->
+  <!-- BEREKENDE POSITIES                                     -->
+  <!-- ====================================================== -->
+  <!-- Midden van het tafelblad boven de vloer -->
+  <xacro:property
+      name="table_top_z"
+      value="${table_leg_height + table_top_thickness / 2.0}"/>
+  <!-- Horizontale posities van de tafelpoten -->
+  <xacro:property
+      name="table_leg_x"
+      value="${table_length / 2.0
+              - table_leg_edge_offset
+              - table_leg_size / 2.0}"/>
+  <xacro:property
+      name="table_leg_y"
+      value="${table_depth / 2.0
+              - table_leg_edge_offset
+              - table_leg_size / 2.0}"/>
+  <!-- Tafelpoot ten opzichte van midden tafelblad -->
+  <xacro:property
+      name="table_leg_relative_z"
+      value="${-(table_top_thickness / 2.0
+                 + table_leg_height / 2.0)}"/>
+  <!-- Steunpoten dicht bij de hoeken van het robotplatform -->
+  <xacro:property
+      name="support_x"
+      value="${platform_length / 2.0 - 0.060}"/>
+  <xacro:property
+      name="support_y"
+      value="${platform_depth / 2.0 - 0.060}"/>
+  <!-- Steunpoten staan direct op het tafelblad -->
+  <xacro:property
+      name="support_relative_z"
+      value="${table_top_thickness / 2.0
+              + support_height / 2.0}"/>
+  <!-- Platform rust op de steunpoten -->
+  <xacro:property
+      name="platform_relative_z"
+      value="${table_top_thickness / 2.0
+              + support_height
+              + platform_thickness / 2.0}"/>
+  <!-- Montageplaat ligt op het platform -->
+  <xacro:property
+      name="mount_plate_relative_z"
+      value="${platform_thickness / 2.0
+              + mount_plate_thickness / 2.0}"/>
+  <!-- ====================================================== -->
+  <!-- MATERIALEN                                             -->
+  <!-- ====================================================== -->
   <material name="brown">
     <color rgba="0.45 0.22 0.08 1.0"/>
   </material>
+  <material name="blue">
+    <color rgba="0.05 0.20 0.80 1.0"/>
+  </material>
+  <material name="dark_grey">
+    <color rgba="0.18 0.18 0.18 1.0"/>
+  </material>
+  <material name="metal_grey">
+    <color rgba="0.60 0.60 0.60 1.0"/>
+  </material>
+  <material name="floor_grey">
+    <color rgba="0.30 0.30 0.30 1.0"/>
+  </material>
+  <!-- ====================================================== -->
+  <!-- HERBRUIKBARE BOX-MACRO                                 -->
+  <!-- ====================================================== -->
+  <xacro:macro
+      name="box_link"
+      params="name size_x size_y size_z material_name">
+    <link name="${name}">
+      <visual>
+        <origin xyz="0 0 0" rpy="0 0 0"/>
+        <geometry>
+          <box size="${size_x} ${size_y} ${size_z}"/>
+        </geometry>
+        <material name="${material_name}"/>
+      </visual>
+      <collision>
+        <origin xyz="0 0 0" rpy="0 0 0"/>
+        <geometry>
+          <box size="${size_x} ${size_y} ${size_z}"/>
+        </geometry>
+      </collision>
+    </link>
+  </xacro:macro>
+  <!-- ====================================================== -->
+  <!-- ROOT EN VLOER                                          -->
+  <!-- ====================================================== -->
   <link name="environment_root"/>
-  <link name="table_top">
-    <visual>
-      <geometry>
-        <box size="1.60 0.80 0.025"/>
-      </geometry>
-      <material name="brown"/>
-    </visual>
-    <collision>
-      <geometry>
-        <box size="1.60 0.80 0.025"/>
-      </geometry>
-    </collision>
-  </link>
+  <xacro:box_link
+      name="floor"
+      size_x="3.0"
+      size_y="3.0"
+      size_z="0.01"
+      material_name="floor_grey"/>
+  <joint name="environment_root_to_floor" type="fixed">
+    <parent link="environment_root"/>
+    <child link="floor"/>
+    <origin xyz="0 0 -0.005" rpy="0 0 0"/>
+  </joint>
+  <!-- ====================================================== -->
+  <!-- TAFELBLAD                                              -->
+  <!-- ====================================================== -->
+  <xacro:box_link
+      name="table_top"
+      size_x="${table_length}"
+      size_y="${table_depth}"
+      size_z="${table_top_thickness}"
+      material_name="brown"/>
   <joint name="environment_root_to_table_top" type="fixed">
     <parent link="environment_root"/>
     <child link="table_top"/>
-    <origin xyz="0 0 0.7375" rpy="0 0 0"/>
+    <origin xyz="0 0 ${table_top_z}" rpy="0 0 0"/>
+  </joint>
+  <!-- ====================================================== -->
+  <!-- VIER TAFELPOTEN                                        -->
+  <!-- ====================================================== -->
+  <xacro:box_link
+      name="table_leg_front_left"
+      size_x="${table_leg_size}"
+      size_y="${table_leg_size}"
+      size_z="${table_leg_height}"
+      material_name="blue"/>
+  <joint name="table_top_to_leg_front_left" type="fixed">
+    <parent link="table_top"/>
+    <child link="table_leg_front_left"/>
+    <origin
+        xyz="${table_leg_x}
+             ${-table_leg_y}
+             ${table_leg_relative_z}"
+        rpy="0 0 0"/>
+  </joint>
+  <xacro:box_link
+      name="table_leg_front_right"
+      size_x="${table_leg_size}"
+      size_y="${table_leg_size}"
+      size_z="${table_leg_height}"
+      material_name="blue"/>
+  <joint name="table_top_to_leg_front_right" type="fixed">
+    <parent link="table_top"/>
+    <child link="table_leg_front_right"/>
+    <origin
+        xyz="${-table_leg_x}
+             ${-table_leg_y}
+             ${table_leg_relative_z}"
+        rpy="0 0 0"/>
+  </joint>
+  <xacro:box_link
+      name="table_leg_back_left"
+      size_x="${table_leg_size}"
+      size_y="${table_leg_size}"
+      size_z="${table_leg_height}"
+      material_name="blue"/>
+  <joint name="table_top_to_leg_back_left" type="fixed">
+    <parent link="table_top"/>
+    <child link="table_leg_back_left"/>
+    <origin
+        xyz="${table_leg_x}
+             ${table_leg_y}
+             ${table_leg_relative_z}"
+        rpy="0 0 0"/>
+  </joint>
+  <xacro:box_link
+      name="table_leg_back_right"
+      size_x="${table_leg_size}"
+      size_y="${table_leg_size}"
+      size_z="${table_leg_height}"
+      material_name="blue"/>
+  <joint name="table_top_to_leg_back_right" type="fixed">
+    <parent link="table_top"/>
+    <child link="table_leg_back_right"/>
+    <origin
+        xyz="${-table_leg_x}
+             ${table_leg_y}
+             ${table_leg_relative_z}"
+        rpy="0 0 0"/>
+  </joint>
+  <!-- ====================================================== -->
+  <!-- STEUNPOTEN OP HET TAFELBLAD                            -->
+  <!-- ====================================================== -->
+  <xacro:box_link
+      name="platform_support_front_left"
+      size_x="${support_size_x}"
+      size_y="${support_size_y}"
+      size_z="${support_height}"
+      material_name="blue"/>
+  <joint name="table_top_to_platform_support_front_left"
+         type="fixed">
+    <parent link="table_top"/>
+    <child link="platform_support_front_left"/>
+    <origin
+        xyz="${support_x}
+             ${-support_y}
+             ${support_relative_z}"
+        rpy="0 0 0"/>
+  </joint>
+  <xacro:box_link
+      name="platform_support_front_right"
+      size_x="${support_size_x}"
+      size_y="${support_size_y}"
+      size_z="${support_height}"
+      material_name="blue"/>
+  <joint name="table_top_to_platform_support_front_right"
+         type="fixed">
+    <parent link="table_top"/>
+    <child link="platform_support_front_right"/>
+    <origin
+        xyz="${-support_x}
+             ${-support_y}
+             ${support_relative_z}"
+        rpy="0 0 0"/>
+  </joint>
+  <xacro:box_link
+      name="platform_support_back_left"
+      size_x="${support_size_x}"
+      size_y="${support_size_y}"
+      size_z="${support_height}"
+      material_name="blue"/>
+  <joint name="table_top_to_platform_support_back_left"
+         type="fixed">
+    <parent link="table_top"/>
+    <child link="platform_support_back_left"/>
+    <origin
+        xyz="${support_x}
+             ${support_y}
+             ${support_relative_z}"
+        rpy="0 0 0"/>
+  </joint>
+  <xacro:box_link
+      name="platform_support_back_right"
+      size_x="${support_size_x}"
+      size_y="${support_size_y}"
+      size_z="${support_height}"
+      material_name="blue"/>
+  <joint name="table_top_to_platform_support_back_right"
+         type="fixed">
+    <parent link="table_top"/>
+    <child link="platform_support_back_right"/>
+    <origin
+        xyz="${-support_x}
+             ${support_y}
+             ${support_relative_z}"
+        rpy="0 0 0"/>
+  </joint>
+  <!-- ====================================================== -->
+  <!-- ROBOTWERKPLATFORM                                      -->
+  <!-- ====================================================== -->
+  <xacro:box_link
+      name="workcell_platform"
+      size_x="${platform_length}"
+      size_y="${platform_depth}"
+      size_z="${platform_thickness}"
+      material_name="dark_grey"/>
+  <joint name="table_top_to_workcell_platform" type="fixed">
+    <parent link="table_top"/>
+    <child link="workcell_platform"/>
+    <origin
+        xyz="0 0 ${platform_relative_z}"
+        rpy="0 0 0"/>
+  </joint>
+  <!-- ====================================================== -->
+  <!-- ROBOTMONTAGEPLAAT                                      -->
+  <!-- ====================================================== -->
+  <xacro:box_link
+      name="robot_mounting_plate"
+      size_x="${mount_plate_length}"
+      size_y="${mount_plate_depth}"
+      size_z="${mount_plate_thickness}"
+      material_name="metal_grey"/>
+  <joint name="workcell_platform_to_mounting_plate"
+         type="fixed">
+    <parent link="workcell_platform"/>
+    <child link="robot_mounting_plate"/>
+    <origin
+        xyz="0 0.235 ${mount_plate_relative_z}"
+        rpy="0 0 0"/>
+  </joint>
+  <!--
+    Referentieframe op de bovenkant van de montageplaat.
+    Hier moet later de officiële Lite 6-base aan gekoppeld worden.
+  -->
+  <link name="robot_mount_frame"/>
+  <joint name="mounting_plate_to_robot_mount_frame"
+         type="fixed">
+    <parent link="robot_mounting_plate"/>
+    <child link="robot_mount_frame"/>
+    <origin
+        xyz="0 0 ${mount_plate_thickness / 2.0}"
+        rpy="0 0 0"/>
+  </joint>
+  <!-- ====================================================== -->
+  <!-- STOEL VOOR DE TAFEL                                    -->
+  <!-- ====================================================== -->
+  <xacro:box_link
+      name="chair_seat"
+      size_x="${chair_width}"
+      size_y="${chair_depth}"
+      size_z="${chair_seat_thickness}"
+      material_name="brown"/>
+  <joint name="environment_root_to_chair_seat" type="fixed">
+    <parent link="environment_root"/>
+    <child link="chair_seat"/>
+    <origin
+        xyz="0
+             -0.80
+             ${chair_leg_height + chair_seat_thickness / 2.0}"
+        rpy="0 0 3.14159"/>
+  </joint>
+  <!-- Stoelpoot linksvoor -->
+  <xacro:box_link
+      name="chair_leg_front_left"
+      size_x="${chair_leg_size}"
+      size_y="${chair_leg_size}"
+      size_z="${chair_leg_height}"
+      material_name="blue"/>
+  <joint name="chair_seat_to_leg_front_left" type="fixed">
+    <parent link="chair_seat"/>
+    <child link="chair_leg_front_left"/>
+    <origin
+        xyz="${chair_width / 2.0 - 0.04}
+             ${-chair_depth / 2.0 + 0.04}
+             ${-(chair_seat_thickness / 2.0
+                + chair_leg_height / 2.0)}"
+        rpy="0 0 0"/>
+  </joint>
+  <!-- Stoelpoot rechtsvoor -->
+  <xacro:box_link
+      name="chair_leg_front_right"
+      size_x="${chair_leg_size}"
+      size_y="${chair_leg_size}"
+      size_z="${chair_leg_height}"
+      material_name="blue"/>
+  <joint name="chair_seat_to_leg_front_right" type="fixed">
+    <parent link="chair_seat"/>
+    <child link="chair_leg_front_right"/>
+    <origin
+        xyz="${-chair_width / 2.0 + 0.04}
+             ${-chair_depth / 2.0 + 0.04}
+             ${-(chair_seat_thickness / 2.0
+                + chair_leg_height / 2.0)}"
+        rpy="0 0 0"/>
+  </joint>
+  <!-- Stoelpoot linksachter -->
+  <xacro:box_link
+      name="chair_leg_back_left"
+      size_x="${chair_leg_size}"
+      size_y="${chair_leg_size}"
+      size_z="${chair_leg_height}"
+      material_name="blue"/>
+  <joint name="chair_seat_to_leg_back_left" type="fixed">
+    <parent link="chair_seat"/>
+    <child link="chair_leg_back_left"/>
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
Commit message: Cartesian bewegeing en beweging functies toegepast

File: src/a2_workcell_description/urdf/workcell.urdf.xacro (robot description, xacro)
@@ -96,4 +96,10 @@
     <color rgba="0.30 0.30 0.30 1.0"/>
   </material>
+    <material name="blocker_red">
+    <color rgba="0.8 0.1 0.1 1.0"/>
+    </material>
+    <material name="standard_gray">
+    <color rgba="0.45 0.45 0.45 1.0"/>
+    </material>
   <!-- ====================================================== -->
   <!-- HERBRUIKBARE BOX-MACRO                                 -->
@@ -427,3 +433,124 @@
         rpy="0 0 0"/>
   </joint>
+    <!-- ========================= -->
+    <!-- Blocker screen assembly   -->
+    <!-- ========================= -->
+    <!--
+    Invisible assembly frame.
+    Move/rotate this frame, and the blocker + standards move together.
+    -->
+    <link name="blocker_assembly_frame"/>
+    <!--
+    Blocker/screen:
+    Real thickness is 0.5 mm, but visualized as 5 mm for RViz visibility.
+    Size:
+    width  = 0.300 m
+    thick  = 0.005 m
+    height = 0.375 m
+    -->
+    <link name="blocker_screen">
+    <visual>
+        <origin xyz="0 0 0" rpy="0 0 0"/>
+        <geometry>
+        <box size="0.300 0.005 0.375"/>
+        </geometry>
+        <material name="blocker_red"/>
+    </visual>
+    <collision>
+        <origin xyz="0 0 0" rpy="0 0 0"/>
+        <geometry>
+        <box size="0.300 0.005 0.375"/>
+        </geometry>
+    </collision>
+    </link>
+   <!--
+    Left standard/support.
+    Reduced length from 10 cm to 8 cm so it does not stick out.
+    Size:
+    length = 0.080 m
+    width  = 0.050 m
+    height = 0.100 m
+    -->
+    <link name="blocker_standard_left">
+    <visual>
+        <origin xyz="0 0 0" rpy="0 0 0"/>
+        <geometry>
+        <box size="0.080 0.050 0.100"/>
+        </geometry>
+        <material name="standard_gray"/>
+    </visual>
+    <collision>
+        <origin xyz="0 0 0" rpy="0 0 0"/>
+        <geometry>
+        <box size="0.080 0.050 0.100"/>
+        </geometry>
+    </collision>
+    </link>
+    <!--
+    Right standard/support.
+    Reduced length from 10 cm to 8 cm.
+    -->
+    <link name="blocker_standard_right">
+    <visual>
+        <origin xyz="0 0 0" rpy="0 0 0"/>
+        <geometry>
+        <box size="0.080 0.050 0.100"/>
+        </geometry>
+        <material name="standard_gray"/>
+    </visual>
+    <collision>
+        <origin xyz="0 0 0" rpy="0 0 0"/>
+        <geometry>
+        <box size="0.080 0.050 0.100"/>
+        </geometry>
+    </collision>
+    </link>
+    <!--
+    Attach the entire blocker assembly to the work platform.
+    x = 0.000 keeps it centered left/right.
+    y = -0.150 places it in the middle/front area of the workspace.
+    yaw = 1.5708 rotates the entire blocker + standards 90 degrees.
+    Because the standards and screen are children of blocker_assembly_frame,
+    they rotate and move together.
+    -->
+    <joint name="blocker_assembly_joint" type="fixed">
+    <parent link="workcell_platform"/>
+    <child link="blocker_assembly_frame"/>
+    <origin xyz="0.000 -0.130 0.000" rpy="0 0 1.5708"/>
+    </joint>
+    <!--
+    Standards sit on top of the work platform.
+    z = platform_half_thickness + standard_half_height
+    z = 0.019/2 + 0.100/2
+    z = 0.0095 + 0.050
+    z = 0.0595
+    -->
+    <joint name="blocker_standard_left_joint" type="fixed">
+    <parent link="blocker_assembly_frame"/>
+    <child link="blocker_standard_left"/>
+    <origin xyz="-0.110 0.000 0.0595" rpy="0 0 0"/>
+    </joint>
+    <joint name="blocker_standard_right_joint" type="fixed">
+    <parent link="blocker_assembly_frame"/>
+    <child link="blocker_standard_right"/>
+    <origin xyz="0.110 0.000 0.0595" rpy="0 0 0"/>
+    </joint>
+    <!--
+    Screen is mounted on top of the standards and sinks into them by about 2.5 cm.
+    Standard top:
+    platform_half_thickness + standard_height
+    0.0095 + 0.100 = 0.1095
+    Screen bottom target:
+    standard_top - 0.025
+    0.1095 - 0.025 = 0.0845
+    Screen center:
+    screen_bottom + screen_height/2
+    0.0845 + 0.375/2
+    0.0845 + 0.1875 = 0.272
+    -->
+    <joint name="blocker_screen_joint" type="fixed">
+    <parent link="blocker_assembly_frame"/>
+    <child link="blocker_screen"/>
+    <origin xyz="0.000 0.000 0.272" rpy="0 0 0"/>
+    </joint>
 </robot>
